Commit message: make descritption file into package

File: ve026a_description/ve026a.urdf (robot description, URDF)
Before this commit: robot ve026a, 8 links, 7 joints
Links:
- link J1: geometry collision mesh filename=package://ve026a_description/J1.dae scale=1 1 1; visual mesh filename=package://ve026a_description/J1.dae scale=1 1 1
- link J2: geometry collision mesh filename=package://ve026a_description/J2.dae scale=1 1 1; visual mesh filename=package://ve026a_description/J2.dae scale=1 1 1
- link J3: geometry collision mesh filename=package://ve026a_description/J3.dae scale=1 1 1; visual mesh filename=package://ve026a_description/J3.dae scale=1 1 1
- link J4: geometry collision mesh filename=package://ve026a_description/J4.dae scale=1 1 1; visual mesh filename=package://ve026a_description/J4.dae scale=1 1 1
- link J5: geometry collision mesh filename=package://ve026a_description/J5.dae scale=1 1 1; visual mesh filename=package://ve026a_description/J5.dae scale=1 1 1
- link J6: geometry collision mesh filename=package://ve026a_description/J6.dae scale=1 1 1; visual mesh filename=package://ve026a_description/J6.dae scale=1 1 1
- link base_link: geometry collision mesh filename=package://ve026a_description/base_link.dae scale=1 1 1; visual mesh filename=package://ve026a_description/base_link.dae scale=1 1 1

Commit message: fixed ve026a.urdf

File: ve026a_description/ve026a.urdf (robot description, URDF)
Before this commit: robot ve026a, 8 links, 7 joints
Joints:
- joint joint_6: axis 0.000000 0.000000 0.000000 -> 0.000000 0.000000 1.000000; origin xyz=0.000000 0.000000 -0.320000 rpy=0.000000 0.000000 0.000000 -> xyz=0.000000 0.000000 0.088 rpy=0.000000 0.000000 0.000000
