Commit message: Add few changes

File: ve026a_description/urdf/ve026a_iman3.urdf (robot description, URDF)
Before this commit: robot ve026a, 10 links, 9 joints
Joints:
- joint joint_5: origin xyz=0.000000 0.000000 0.090000 rpy=0.000000 0.000000 0.000000 -> xyz=0.000000 0.000000 0.070000 rpy=0.000000 0.000000 0.000000
